File: lora_projesi/verici/verici.kicad_sch (KiCad schematic)
At the start: 37 parts, among them J1 USB-C, J2 SMA, SW1 ANA ACMA-KAPAMA, SW2 DUGME 1, SW3 DUGME 2, SW4 DUGME 3, SW5 DUGME 4, SW6 DUGME 5, SW7 DUGME 6, U1 ESP32-S3-WROOM-1-N4, U2 TPS63031DSKR, U3 USBLC6-2SC6, U4 RFM95W-915S2

Commit message: A7670SA, Ra-01H, LM66100 ideal diyot, SRP7028A, USBLC6-2: uretec ve kutuphane (kart yonlendirmesi suruyor)
Co-Authored-By: Claude Sonnet 5.5 <noreply@anthropic.com>
Claude-Session: https://claude.ai/code/session_01Q71gHQtKJ86ZE2CtYTYSwP
Parts:
- removed U4: RFM95W-915S2, RF_Module:HOPERF_RFM9XW_SMD, symbol RF_Module:RFM95W-915S2
- added U4: Ra-01H, Ozel:Ra-01H, symbol Ozel:Ra-01H
Connections:
- net +3V3: now also U4.3 (VDD)
- net ANT_RF: now also U4.1 (ANT)
- net GND: now also U4.16 (GND), U4.2 (GND), U4.9 (GND)
- net LORA_DIO0: now also U4.5 (DIO0)
- net LORA_DIO1: now also U4.6 (DIO1)
- net LORA_MISO: now also U4.13 (MISO)
- net LORA_MOSI: now also U4.14 (MOSI)
- net LORA_NSS: now also U4.15 (NSS)
- net LORA_RESET: now also U4.4 (RESET)
- net LORA_SCK: now also U4.12 (SCK)
Other:
- note added: "LoRa: Ra-01H (SX1276) ve anten konnektoru"
- note removed: "LoRa: RFM95W-915S2 ve anten konnektoru"
