File: lora_projesi/verici/verici_once.kicad_pcb (KiCad board)
At the start: 4 copper layers, 40 x 100 mm, 39 parts, among them J1 USB-C, J2 SMA, SW1 ANA ACMA-KAPAMA, SW2 DUGME 1, SW3 DUGME 2, SW4 DUGME 3, SW5 DUGME 4, SW6 DUGME 5, SW7 DUGME 6, U1 ESP32-S3-WROOM-1-N4, U2 TPS63031DSKR, U3 USBLC6-2SC6, U4 RFM95W-915S2

Commit message: Verici: 4 katmanli kart, DRC temiz, uretim dosyalari, tasarim notu
Co-Authored-By: Claude Sonnet 5.5 <noreply@anthropic.com>
Claude-Session: https://claude.ai/code/session_01Q71gHQtKJ86ZE2CtYTYSwP
Parts:
- moved U3 12.1 mm to (37.0, 15.0)
- moved J1 1.00 mm to (31.0, 4.20)

Commit message: A7670SA, Ra-01H, LM66100 ideal diyot, SRP7028A, USBLC6-2: uretec ve kutuphane (kart yonlendirmesi suruyor)
Co-Authored-By: Claude Sonnet 5.5 <noreply@anthropic.com>
Claude-Session: https://claude.ai/code/session_01Q71gHQtKJ86ZE2CtYTYSwP
Parts:
- U4: value RFM95W-915S2 -> Ra-01H; footprint HOPERF_RFM9XW_SMD -> Ra-01H
- moved R9 5.49 mm to (26.6, 11.0)
- moved R10 5.24 mm to (26.6, 13.5)
- moved C9 4.50 mm to (5.00, 18.0)
- moved C8 4.00 mm to (5.00, 13.0)
- moved U4 3.30 mm to (14.6, 17.2), turned to 0 degrees
Connections:
- U4 pad 1: GND -> ANT_RF
- U4 pad 10: GND -> (no net)
- U4 pad 12: (no net) -> LORA_SCK
- U4 pad 13: +3V3 -> LORA_MISO
- U4 pad 14: LORA_DIO0 -> LORA_MOSI
- U4 pad 15: LORA_DIO1 -> LORA_NSS
- U4 pad 16: (no net) -> GND
- U4 pad 2: LORA_MISO -> GND
- U4 pad 3: LORA_MOSI -> +3V3
- U4 pad 4: LORA_SCK -> LORA_RESET
- U4 pad 5: LORA_NSS -> LORA_DIO0
- U4 pad 6: LORA_RESET -> LORA_DIO1
- U4 pad 8: GND -> (no net)
- U4 pad 9: ANT_RF -> GND
Routing:
- net ANT_RF: track 9.00 -> 5.70 mm
